Commit message: for jackal

File: zed_wrapper/urdf/zed.urdf (robot description, URDF)
Before this commit: robot zed_camera, 6 links, 5 joints
Links:
- removed link base_link
- added link front_mount
Joints:
- joint zed_camera_center_joint: parent base_link -> front_mount

Commit message: update

File: zed_wrapper/urdf/zed.urdf (robot description, URDF)
Before this commit: robot zed_camera, 6 links, 5 joints
Links:
- removed link front_mount
- added link mid_mount
Joints:
- joint zed_camera_center_joint: origin xyz=0 0 0 rpy=0 0 0 -> xyz=0 0 0.47 rpy=0 0 0; parent front_mount -> mid_mount

Commit message: update

File: zed_wrapper/urdf/zed.urdf (robot description, URDF)
Before this commit: robot zed_camera, 6 links, 5 joints
Joints:
- joint zed_camera_center_joint: origin xyz=0 0 0.47 rpy=0 0 0 -> xyz=-0.02 0 0.33 rpy=0 0 0
